File: hardware/led_ceiling_light.kicad_sch (KiCad schematic)
At the start: 28 parts, among them J1 Screw_Terminal_01x03, Q1 BSS123, U1 AL8861

Commit message: Fix D13 footprint
Parts:
- D13: footprint Diode_SMD:D_SC-80_HandSoldering -> Diode_SMD:D_MiniMELF_Handsoldering
Changed lines of the file:
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@@
       (effects (font (size 1.27 1.27)) (justify left))
     )
-    (property "Footprint" "Diode_SMD:D_SC-80_HandSoldering" (id 2) (at 100.33 100.33 0)
+    (property "Footprint" "Diode_SMD:D_MiniMELF_Handsoldering" (id 2) (at 100.33 100.33 0)
       (effects (font (size 1.27 1.27)) hide)
     )
@@
     )
     (path "/591c7a48-6647-47f5-be47-c2508213f188"
-      (reference "D13") (unit 1) (value "2.7V") (footprint "Diode_SMD:D_SC-80_HandSoldering")
+      (reference "D13") (unit 1) (value "2.7V") (footprint "Diode_SMD:D_MiniMELF_Handsoldering")
     )
     (path "/bf06e978-418f-42d7-bbde-c8a97f9d162c"
